File: kicad_projects/led_flasher/led_flasher.kicad_pcb (KiCad board)
At the start: 2 copper layers, 80 x 50 mm, 17 parts, among them Q1 2N3904, Q2 2N3904, SW1 SW_SPDT

Commit message: kicad logo footprints updated
Parts:
- moved G*** 2.50 mm to (213.5, 88.0)
