File: kicad_projects/motor_control/motor_control.kicad_pcb (KiCad board)
At the start: 2 copper layers, 110 x 65 mm, 36 parts, among them J1 Conn_01x02_Pin, J2 Conn_01x02_Pin, Q1 Q_NMOS_GDS, Q2 Q_NMOS_GDS, Q3 Q_NMOS_GDS, Q4 Q_NMOS_GDS, U1 40106, U2 LM3914N

Commit message: route traces added but there is thermal relief error
Parts:
- moved Q1 52.1 mm to (152.6, 65.0)
- moved J2 46.1 mm to (163.5, 68.2)
- moved Q2 40.9 mm to (152.6, 74.0)
- moved Q4 36.6 mm to (152.6, 94.0)
- moved Q3 34.4 mm to (152.6, 84.0)
- moved U1 30.1 mm to (132.4, 67.4)
- moved D2 28.1 mm to (154.0, 102.0), turned to -90 degrees
- moved D1 28.0 mm to (146.0, 102.2), turned to -90 degrees
- moved RV2 27.2 mm to (135.0, 112.5)
- moved RV1 27.1 mm to (135.0, 97.5)
- moved D6 26.7 mm to (154.0, 114.0), turned to -90 degrees
- moved D5 26.4 mm to (146.0, 114.0), turned to -90 degrees
- moved J1 24.6 mm to (163.9, 84.0)
- moved D4 10.5 mm to (162.0, 102.0), turned to -90 degrees
- moved R12 7.42 mm to (170.0, 105.0), turned to -90 degrees
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Routing:
- net VDD: track 0.00 -> 475.2 mm
- net Net-(C1-Pad1): track 0.00 -> 197.2 mm
- net Net-(D2-K): track 0.00 -> 160.3 mm
- net Net-(U2-REFOUT): track 0.00 -> 146.5 mm
- net Net-(C2-Pad1): track 0.00 -> 113.8 mm, vias 0 -> 2
- net Net-(Q3-G): track 0.00 -> 110.3 mm
- net Net-(D3-A): track 0.00 -> 104.0 mm
- net Net-(D4-A): track 0.00 -> 77.6 mm
- net Net-(D5-K): track 0.00 -> 73.9 mm
- net Net-(D1-K): track 0.00 -> 51.3 mm
- net Net-(U2-SIG): track 0.00 -> 48.9 mm
- net Net-(Q1-G): track 0.00 -> 46.0 mm
- net Net-(Q2-G): track 0.00 -> 41.5 mm, vias 0 -> 2
- net Net-(Q1-D): track 0.00 -> 26.7 mm
- net Net-(D6-K): track 0.00 -> 23.5 mm
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
Commit message: route traces fixed
Parts:
- added G***: LOGO, logos:pig, F.Cu at (215.0, 113.0)
- moved R1 27.3 mm to (175.9, 117.0)
- moved D5 16.9 mm to (162.4, 118.0), turned to 0 degrees
- moved D1 9.03 mm to (148.0, 111.0), turned to 0 degrees
- moved R12 7.75 mm to (175.9, 110.0), turned to 0 degrees
- moved D6 7.05 mm to (148.2, 118.0), turned to 0 degrees
- moved D2 6.32 mm to (148.0, 104.0), turned to 0 degrees
- moved J1 5.00 mm to (163.9, 89.0)
- moved J2 3.86 mm to (163.9, 72.0)
- moved Q1 3.00 mm to (152.6, 68.0)
- moved Q2 3.00 mm to (152.6, 77.0)
- moved D3 2.22 mm to (162.4, 111.0), turned to 0 degrees
- moved D4 2.04 mm to (162.4, 104.0), turned to 0 degrees
- moved Q3 2.00 mm to (152.6, 86.0)
- moved U2 1.08 mm to (178.0, 68.3)
- moved Q4 1.05 mm to (152.6, 95.0)
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Routing:
- net VDD: track 475.2 -> 101.0 mm, vias 0 -> 6
- net Net-(D2-K): track 160.3 -> 19.3 mm
- net Net-(U2-REFOUT): track 146.5 -> 27.3 mm
- net Net-(Q3-G): track 110.3 -> 22.2 mm
- net Net-(C1-Pad1): track 197.2 -> 114.1 mm
- net Net-(Q2-G): track 41.5 -> 101.5 mm
- net Net-(D3-A): track 104.0 -> 76.5 mm
- net Net-(D5-A): track 14.7 -> 37.2 mm
- net Net-(D4-A): track 77.6 -> 55.3 mm
- net Net-(C2-Pad1): track 113.8 -> 93.4 mm, vias 2 -> 4
- net Net-(Q1-G): track 46.0 -> 27.1 mm
- net Net-(Q1-D): track 26.7 -> 10.1 mm
- net Net-(D5-K): track 73.9 -> 62.0 mm, vias 0 -> 4
- net Net-(D1-K): track 51.3 -> 62.1 mm
- net Net-(D1-A): track 16.8 -> 26.2 mm
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Other:
- board text added: "Motor Controller Catharine Zhou"
